File: ATX-breakout.kicad_pcb (KiCad board)
At the start: 2 copper layers, 67 x 59.5 mm, 24 parts, among them J1 I2C, J10 3V3 out, J11 12V out, J12 12V out, J2 EPS, J3 USB_A, J4 Raspberry_Pi_2_3, J5 ATX24pin, J6 12V out, J7 pson ext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

Commit message: Added mounting holes
Parts:
- removed the G*** at (69.0, 87.2) (x2)
- added G***: LOGO, graphics:kiwi, B.Cu at (19.0, 45.7)
- added G***: LOGO, graphics:kiwi, F.Cu at (19.0, 45.7)
- added REF**: MountingHole_3.2mm_M3_DIN965, MountingHole:MountingHole_3.2mm_M3_DIN965, F.Cu at (3.92, 55.6)
- added REF**: MountingHole_3.2mm_M3_DIN965, MountingHole:MountingHole_3.2mm_M3_DIN965, F.Cu at (64.0, 56.5)
- added REF**: MountingHole_3.2mm_M3_DIN965, MountingHole:MountingHole_3.2mm_M3_DIN965, F.Cu at (19.0, 18.5)
- moved J5 68.3 mm to (3.30, 29.9)
- moved JP3 68.3 mm to (36.4, 42.4)
- moved R2 68.3 mm to (40.4, 50.9)
- moved R5 68.3 mm to (50.2, 50.9)
- moved J1 68.3 mm to (61.5, 32.3)
- moved J10 68.3 mm to (11.1, 6.80)
- moved J11 68.3 mm to (63.1, 6.80)
- moved J12 68.3 mm to (58.0, 19.2)
- moved J2 68.3 mm to (50.0, 19.6)
- moved J3 68.3 mm to (12.0, 14.8)
- moved J4 68.3 mm to (57.1, 54.3)
- moved J6 68.3 mm to (50.1, 6.80)
- moved J7 68.3 mm to (40.9, 45.6)
- moved J8 68.3 mm to (24.1, 6.80)
- moved J9 68.3 mm to (37.1, 6.80)
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Routing:
- net GND: track 113.3 -> 124.2 mm
- net +3V3: track 96.6 -> 100.8 mm
- net +12V: track 33.7 -> 37.4 mm
- net +5V: track 89.0 -> 92.1 mm
- net Net-(J3-Pad1): track 18.0 -> 21.0 mm
- net /5v_rpi: track 40.6 -> 40.0 mm
Other:
- board text added: "(0,0)"
- board text added: "(19, 18.5)"
- board text added: "(3.92, 55.57)"
- board text added: "(64, 56.5)"
- board text added: "(x,y)"
- board text added: "x"
- board text added: "y"
